File: kicad-example/kicad-example.kicad_pcb (KiCad board)
At the start: 2 copper layers, 20 x 16 mm, 7 parts, among them U1 TL072

Commit message: Route
Routing:
- net Net-(R1-Pad2): track 0.00 -> 5.73 mm
- net OUT_A: track 0.00 -> 2.85 mm
Changed lines of the file:
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@@
   )
   (gr_rect (start 126 53) (end 146 69) (layer "Edge.Cuts") (width 0.1) (fill none))
+  (segment (start 130 56) (end 130 59) (width 0.25) (layer "F.Cu") (net 5))
+  (segment (start 130.985 59.985) (end 132.32 59.985) (width 0.25) (layer "F.Cu") (net 5))
+  (segment (start 130 59) (end 130.985 59.985) (width 0.25) (layer "F.Cu") (net 5))
+  (segment (start 132.32 56.32) (end 132 56) (width 0.25) (layer "F.Cu") (net 8))
+  (segment (start 132.32 58.715) (end 132.32 56.32) (width 0.25) (layer "F.Cu") (net 8))
 )

Commit message: Workflow
Routing:
- added copper zone on B.Cu, net GND
Changed lines of the file:
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@@
   (segment (start 132.32 56.32) (end 132 56) (width 0.25) (layer "F.Cu") (net 8))
   (segment (start 132.32 58.715) (end 132.32 56.32) (width 0.25) (layer "F.Cu") (net 8))
+  (zone (net 2) (net_name "GND") (layer "B.Cu") (hatch edge 0.508)
+    (connect_pads (clearance 0.508))
+    (min_thickness 0.254) (filled_areas_thickness no)
+    (fill yes (thermal_gap 0.508) (thermal_bridge_width 0.508))
+    (polygon
+      (pts
+        (xy 147 70)
+        (xy 125 70)
+        (xy 125 52)
+        (xy 147 52)
+      )
+    )
+  )
 )
