File: kicad-example/kicad-example.kicad_sch (KiCad schematic)
At the start: 7 parts, among them U1 TL072

Commit message: Schematic file path
Parts:
- C1, C2: value 10u -> 100n
Changed lines of the file:
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@@
       (effects (font (size 1.27 1.27)) (justify left))
     )
-    (property "Value" "10u" (id 1) (at 119.38 44.4562 0)
+    (property "Value" "100n" (id 1) (at 119.38 44.4562 0)
       (effects (font (size 1.27 1.27)) (justify left))
     )
@@
       (effects (font (size 1.27 1.27)) (justify left))
     )
-    (property "Value" "10u" (id 1) (at 119.38 60.9662 0)
+    (property "Value" "100n" (id 1) (at 119.38 60.9662 0)
       (effects (font (size 1.27 1.27)) (justify left))
     )
@@
     )
     (path "/555653a9-b2be-4b79-97c0-61cfdc9e78e8"
-      (reference "C1") (unit 1) (value "10u") (footprint "Capacitor_SMD:C_0805_2012Metric_Pad1.18x1.45mm_HandSolder")
+      (reference "C1") (unit 1) (value "100n") (footprint "Capacitor_SMD:C_0805_2012Metric_Pad1.18x1.45mm_HandSolder")
     )
     (path "/b66c8b20-cbc1-4d28-abc7-ad990ea20187"
-      (reference "C2") (unit 1) (value "10u") (footprint "Capacitor_SMD:C_0805_2012Metric_Pad1.18x1.45mm_HandSolder")
+      (reference "C2") (unit 1) (value "100n") (footprint "Capacitor_SMD:C_0805_2012Metric_Pad1.18x1.45mm_HandSolder")
     )
     (path "/cd3851c8-43a7-44ba-a57d-7da51bf4d405"

Commit message: Workflow
Connections:
- net VDD: now also U1.8 (V+); no longer U1.4 (V-)
- net VSS: now also U1.4 (V-); no longer U1.8 (V+)
Changed lines of the file:
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@@
+    (pin "1")
+  )
+  (symbol (lib_id "power:PWR_FLAG") (at 240.03 172.72 180) (unit 1)
+    (in_bom yes) (on_board yes) (fields_autoplaced)
+    (property "Reference" "#FLG0101" (id 0) (at 240.03 174.625 0)
+      (effects (font (size 1.27 1.27)) hide)
+    )
+    (property "Value" "PWR_FLAG" (id 1) (at 242.57 173.9899 0)
+      (effects (font (size 1.27 1.27)) (justify right))
+    )
+    (property "Footprint" "" (id 2) (at 240.03 172.72 0)
+      (effects (font (size 1.27 1.27)) hide)
+    )
+    (property "Datasheet" "~" (id 3) (at 240.03 172.72 0)
+      (effects (font (size 1.27 1.27)) hide)
+    )
+    (pin "1")
+  )
+  (symbol (lib_id "power:VDD") (at 240.03 172.72 0) (unit 1)
+    (in_bom yes) (on_board yes)
+    (property "Reference" "#PWR0107" (id 0) (at 240.03 176.53 0)
+      (effects (font (size 1.27 1.27)) hide)
+    )
+    (property "Value" "VDD" (id 1) (at 240.03 168.91 0))
+    (property "Footprint" "" (id 2) (at 240.03 172.72 0)
+      (effects (font (size 1.27 1.27)) hide)
+    )
+    (property "Datasheet" "" (id 3) (at 240.03 172.72 0)
+      (effects (font (size 1.27 1.27)) hide)
+    )
     (pin "1")
   )
@@
     (pin "3")
   )
+  (symbol (lib_id "power:PWR_FLAG") (at 255.27 172.72 0) (unit 1)
+    (in_bom yes) (on_board yes) (fields_autoplaced)
+    (property "Reference" "#FLG0102" (id 0) (at 255.27 170.815 0)
+      (effects (font (size 1.27 1.27)) hide)
+    )
+    (property "Value" "PWR_FLAG" (id 1) (at 257.81 171.4499 0)
+      (effects (font (size 1.27 1.27)) (justify left))
+    )
+    (property "Footprint" "" (id 2) (at 255.27 172.72 0)
+      (effects (font (size 1.27 1.27)) hide)
+    )
+    (property "Datasheet" "~" (id 3) (at 255.27 172.72 0)
+      (effects (font (size 1.27 1.27)) hide)
+    )
+    (pin "1")
+  )
   (symbol (lib_id "Device:R") (at 78.74 63.5 90) (unit 1)
     (in_bom yes) (on_board yes)
@@
     (pin "1")
   )
+  (symbol (lib_id "power:PWR_FLAG") (at 270.51 172.72 0) (unit 1)
+    (in_bom yes) (on_board yes) (fields_autoplaced)
+    (property "Reference" "#FLG?" (id 0) (at 270.51 170.815 0)
+      (effects (font (size 1.27 1.27)) hide)
+    )
+    (property "Value" "PWR_FLAG" (id 1) (at 273.05 171.4499 0)
+      (effects (font (size 1.27 1.27)) (justify left))
+    )
+    (property "Footprint" "" (id 2) (at 270.51 172.72 0)
+      (effects (font (size 1.27 1.27)) hide)
+    )
+    (property "Datasheet" "~" (id 3) (at 270.51 172.72 0)
+      (effects (font (size 1.27 1.27)) hide)
+    )
+    (pin "1")
+  )
   (symbol (lib_id "Amplifier_Operational:TL072") (at 77.47 73.66 0) (mirror x) (unit 2)
     (in_bom yes) (on_board yes)
@@
     (pin "7")
   )
+  (symbol (lib_id "power:GND") (at 270.51 172.72 0) (unit 1)
+    (in_bom yes) (on_board yes)
+    (property "Reference" "#PWR?" (id 0) (at 270.51 179.07 0)
+      (effects (font (size 1.27 1.27)) hide)
+    )
+    (property "Value" "GND" (id 1) (at 270.51 176.53 0))
+    (property "Footprint" "" (id 2) (at 270.51 172.72 0)
+      (effects (font (size 1.27 1.27)) hide)
+    )
+    (property "Datasheet" "" (id 3) (at 270.51 172.72 0)
+      (effects (font (size 1.27 1.27)) hide)
+    )
+    (pin "1")
+  )
   (symbol (lib_id "power:VDD") (at 109.22 39.37 0) (unit 1)
     (in_bom yes) (on_board yes) (fields_autoplaced)
@@
     (pin "2")
   )
-  (symbol (lib_id "Amplifier_Operational:TL072") (at 111.76 48.26 0) (mirror x) (unit 3)
+  (symbol (lib_id "Amplifier_Operational:TL072") (at 111.76 48.26 0) (unit 3)
     (in_bom yes) (on_board yes)
     (property "Reference" "U1" (id 0) (at 104.14 48.26 0))
@@
     (pin "8")
   )
+  (symbol (lib_id "power:VSS") (at 255.27 172.72 180) (unit 1)
+    (in_bom yes) (on_board yes)
+    (property "Reference" "#PWR0108" (id 0) (at 255.27 168.91 0)
+      (effects (font (size 1.27 1.27)) hide)
+    )
+    (property "Value" "VSS" (id 1) (at 254 176.53 0)
+      (effects (font (size 1.27 1.27)) (justify right))
+    )
+    (property "Footprint" "" (id 2) (at 255.27 172.72 0)
+      (effects (font (size 1.27 1.27)) hide)
+    )
+    (property "Datasheet" "" (id 3) (at 255.27 172.72 0)
+      (effects (font (size 1.27 1.27)) hide)
+    )
+    (pin "1")
+  )
   (sheet_instances
     (path "/" (page "1"))
   )
   (symbol_instances
+    (path "/42d7e36f-ba63-4bf8-a540-78fb26027164"
+      (reference "#FLG0101") (unit 1) (value "PWR_FLAG") (footprint "")
+    )
+    (path "/66ac6d1a-c014-49ee-9cee-5b2dc73c2c4d"
+      (reference "#FLG0102") (unit 1) (value "PWR_FLAG") (footprint "")
+    )
+    (path "/98f217f0-09d6-4bf5-a46a-4667b74840e6"
+      (reference "#FLG?") (unit 1) (value "PWR_FLAG") (footprint "")
+    )
     (path "/b9b8c0b1-ada1-40c3-83cc-376afde39596"
       (reference "#PWR0101") (unit 1) (value "GND") (footprint "")
@@
       (reference "#PWR0106") (unit 1) (value "GND") (footprint "")
     )
+    (path "/433fde44-349b-4e9a-bda2-04085147b6fa"
+      (reference "#PWR0107") (unit 1) (value "VDD") (footprint "")
+    )
+    (path "/fb82b49b-a6b7-4a06-ac71-b39da799a8ff"
+      (reference "#PWR0108") (unit 1) (value "VSS") (footprint "")
+    )
+    (path "/aeba8933-d424-4ca4-a8d8-ddffbf74b385"
+      (reference "#PWR?") (unit 1) (value "GND") (footprint "")
+    )
     (path "/555653a9-b2be-4b79-97c0-61cfdc9e78e8"
